File: feather-SAMD21&WD.kicad_pcb (KiCad board)
At the start: 4 copper layers, 51.6 x 22.9 mm, 69 parts, among them J1 JumperSET0, J10 monostable bypass jumper, J2 JumperSET1, J3 JumperSET2, J4 left_header, J5 right_header, J6 Batt_header, J7 reset_enable, J8 16P_USB_C, J9 wd_pwr_jumper, SW1 SW_Push, U2 USBLC6-2SC6, U3 ATSAMD21G18A-M, U4 AP2112K-3.3, U5 MCP73832-2-OT, U6 AP2112K-3.3, X1 32.768

Commit message: finishing touches
Parts:
- removed the G*** at (119.8, 110.1)
- removed the G*** at (120.0, 110.8)
- removed the G*** at (100.8, 106.5)
- moved 3.3wd 0.71 mm to (155.4, 85.3)
- moved C9 0.24 mm to (114.6, 77.2)
Routing:
- net VBUS: track 32.4 -> 37.0 mm
- net ~{RESET}: track 60.6 -> 59.9 mm
- net GND: track 100.9 -> 101.6 mm, vias 20 -> 27
Other:
- board text removed: "3.3"
- board text removed: "59 4F 47 20 57 4D 4B 43"

Commit message: minor changes
Parts:
- C2: value C_Small -> 100n
- C6, C7: value 22pf -> 12.5pf
- D3: value D_Schottky -> D_Schottky(BAT43W)
- WD: value MAX6369 -> MAX6373
- renumbered McuLED to D6, RESET to TP1, WDO to TP2, BattADC to TP3, 3.3wd to TP4, Disch to TP5, 3.3μC to TP6, Thresh to TP7, LdoEN to TP8, 555 to U7
Routing:
- net Net-(U7-DISCH): track 5.29 -> 4.37 mm
Changed lines of the file:
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@@
 		(capping no)
 		(filling no)
-		(zone_defaults)
 		(pcbplotparams
 			(layerselection 0x00000000_00000000_55555555_5755f5ff)
@@
 			)
 		)
-		(property "Value" "MAX6369"
+		(property "Value" "MAX6373"
 			(at 1.4 2.3 0)
 			(layer "F.Fab")
@@
 		(descr "VSSOP, 8 Pin (https://www.jedec.org/standards-documents/docs/mo-187-f)")
 		(tags "VSSOP SO JEDEC-MO-187-AA Texas_DGK0008A")
-		(property "Reference" "555"
+		(property "Reference" "U7"
 			(at 0 0 0)
 			(layer "F.SilkS")
@@
 		(descr "LED SMD 0805 (2012 Metric), square (rectangular) end terminal, IPC-7351 nominal, (Body size source: https://docs.google.com/spreadsheets/d/1BsfQQcO9C6DZCsRaXUlFlo91Tg2WpOkGARC1WS5S8t0/edit?usp=sharing)")
 		(tags "LED handsolder")
-		(property "Reference" "McuLED"
+		(property "Reference" "D6"
 			(at 3.8325 -0.475 0)
 			(layer "F.SilkS")
@@
 			)
 		)
-		(property "Value" "22pf"
+		(property "Value" "12.5pf"
 			(at 0 1.679999 0)
 			(layer "F.Fab")
@@
 			)
 		)
-		(property "Value" "22pf"
+		(property "Value" "12.5pf"
 			(at 0 1.679999 0)
 			(layer "F.Fab")
@@
 			)
 		)
-		(property "Value" "D_Schottky"
+		(property "Value" "D_Schottky(BAT43W)"
 			(at -0.1 1.9 90)
 			(layer "F.Fab")
@@
 			)
 		)
-		(property "Value" "C_Small"
+		(property "Value" "100n"
 			(at 0 1.679999 90)
 			(layer "F.Fab")
@@
 		(descr "SMD pad as test Point, diameter 1.5mm")
 		(tags "test point SMD pad")
-		(property "Reference" "3.3wd"
+		(property "Reference" "TP4"
 			(at -0.085 -1.955 180)
 			(unlocked yes)
@@
 		(descr "SMD pad as test Point, diameter 1.5mm")
 		(tags "test point SMD pad")
-		(property "Reference" "BattADC"
+		(property "Reference" "TP3"
 			(at 0.3 1.725 180)
 			(unlocked yes)
@@
 		(descr "SMD pad as test Point, diameter 1.5mm")
 		(tags "test point SMD pad")
-		(property "Reference" "WDO"
+		(property "Reference" "TP2"
 			(at 0.2 -1.925 180)
 			(unlocked yes)
@@
 		(descr "SMD pad as test Point, diameter 1.5mm")
 		(tags "test point SMD pad")
-		(property "Reference" "RESET"
+		(property "Reference" "TP1"
 			(at 0 1.648 180)
 			(unlocked yes)
@@
 		(descr "SMD pad as test Point, diameter 1.5mm")
 		(tags "test point SMD pad")
-		(property "Reference" "3.3μC"
+		(property "Reference" "TP6"
 			(at -0.325 1.6 180)
 			(unlocked yes)
@@
 		(descr "SMD pad as test Point, diameter 1.5mm")
 		(tags "test point SMD pad")
-		(property "Reference" "LdoEN"
+		(property "Reference" "TP8"
 			(at 0.015 1.845 180)
 			(unlocked yes)
@@
 		(descr "SMD pad as test Point, diameter 1.5mm")
 		(tags "test point SMD pad")
-		(property "Reference" "Thresh"
+		(property "Reference" "TP7"
 			(at -3.05 -0.675 180)
 			(unlocked yes)
@@
 		(descr "SMD pad as test Point, diameter 1.5mm")
 		(tags "test point SMD pad")
-		(property "Reference" "Disch"
+		(property "Reference" "TP5"
 			(at 2.75 0.275 180)
 			(unlocked yes)
@@
 	)
 	(segment
+		(start 125.19 86.88)
+		(end 125.4925 86.88)
+		(width 0.252)
+		(layer "F.Cu")
+		(net "GND")
+	)
+	(segment
 		(start 148.3525 88.555)
 		(end 147.690001 88.555)
@@
 	)
 	(segment
+		(start 122.29 86.73)
+		(end 122.52 86.96)
+		(width 0.252)
+		(layer "F.Cu")
+		(net "GND")
+	)
+	(segment
 		(start 111.6575 75.8825)
 		(end 110 77.54)
@@
 	)
 	(segment
+		(start 122.52 86.96)
+		(end 125.11 86.96)
+		(width 0.252)
+		(layer "F.Cu")
+		(net "GND")
+	)
+	(segment
 		(start 133.42 87.449999)
 		(end 133.420001 87.449999)
@@
 	)
 	(segment
+		(start 125.11 86.96)
+		(end 125.19 86.88)
+		(width 0.252)
+		(layer "F.Cu")
+		(net "GND")
+	)
+	(segment
 		(start 157.48 85.8)
 		(end 157.48 83.95)
@@
 	)
 	(segment
-		(start 125.11 86.96)
-		(end 122.54 86.96)
-		(width 0.252)
-		(layer "F.Cu")
-		(net "GND")
-	)
-	(segment
 		(start 123.69 79.89)
 		(end 125.02 81.22)
@@
 	)
 	(segment
-		(start 125.19 86.88)
-		(end 125.11 86.96)
-		(width 0.252)
-		(layer "F.Cu")
-		(net "GND")
-	)
-	(segment
 		(start 147.19 88.054999)
 		(end 147.19 87.999297)
@@
 	)
 	(segment
-		(start 125.4925 86.88)
-		(end 125.19 86.88)
-		(width 0.252)
-		(layer "F.Cu")
-		(net "GND")
-	)
-	(segment
 		(start 152.72 92.3)
 		(end 153.67 93.25)
@@
 	)
 	(via
-		(at 122.54 86.96)
+		(at 122.29 86.73)
 		(size 0.6)
 		(drill 0.3)
@@
 	)
 	(segment
-		(start 149.75 80.54)
-		(end 149.1 79.89)
-		(width 0.252)
-		(layer "B.Cu")
-		(net "Net-(U7-DISCH)")
-	)
-	(segment
 		(start 116.93 77.9575)
 		(end 117.0575 77.9575)
@@
 	)
 	(segment
-		(start 118.175 86.639998)
-		(end 118.5375 86.639998)
+		(start 122.910665 85.27)
+		(end 126.468198 85.27)
 		(width 0.2)
 		(layer "F.Cu")
@@
 	)
 	(segment
-		(start 118.5375 86.639998)
-		(end 119.907498 85.27)
+		(start 122.410665 85.27)
+		(end 122.910665 85.27)
 		(width 0.2)
 		(layer "F.Cu")
@@
 	)
 	(segment
-		(start 128.538198 83.2)
-		(end 131.441802 83.2)
+		(start 118.407501 86.589999)
+		(end 117.9975 86.589999)
 		(width 0.2)
 		(layer "F.Cu")
@@
 	)
 	(segment
-		(start 118.407501 86.589999)
-		(end 117.9975 86.589999)
+		(start 119.907498 85.27)
+		(end 121.770665 85.27)
 		(width 0.2)
 		(layer "F.Cu")
@@
 	)
 	(segment
-		(start 126.468198 85.27)
-		(end 128.538198 83.2)
+		(start 122.170665 85.51)
+		(end 122.410665 85.27)
 		(width 0.2)
 		(layer "F.Cu")
@@
 	)
 	(segment
-		(start 119.907498 85.27)
-		(end 126.468198 85.27)
+		(start 118.5375 86.639998)
+		(end 119.907498 85.27)
+		(width 0.2)
+		(layer "F.Cu")
+		(net "D+")
+	)
+	(segment
+		(start 122.010665 85.51)
+		(end 122.170665 85.51)
+		(width 0.2)
+		(layer "F.Cu")
+		(net "D+")
+	)
+	(segment
+		(start 121.770665 85.27)
+		(end 122.010665 85.51)
 		(width 0.2)
 		(layer "F.Cu")
@@
 	)
 	(segment
+		(start 128.538198 83.2)
+		(end 131.441802 83.2)
+		(width 0.2)
+		(layer "F.Cu")
+		(net "D+")
+	)
+	(segment
+		(start 118.175 86.639998)
+		(end 118.5375 86.639998)
+		(width 0.2)
+		(layer "F.Cu")
+		(net "D+")
+	)
+	(segment
+		(start 126.468198 85.27)
+		(end 128.538198 83.2)
+		(width 0.2)
+		(layer "F.Cu")
+		(net "D+")
+	)
+	(segment
 		(start 131.670002 83.699999)
 		(end 131.695002 83.674999)
@@
 	)
 	(segment
-		(start 113.625998 87.135687)
-		(end 115.404311 87.135687)
+		(start 112.679998 86.392509)
+		(end 112.93682 86.135687)
 		(width 0.252)
 		(layer "F.Cu")
@@
 	)
 	(segment
-		(start 112.679998 86.392509)
-		(end 112.93682 86.135687)
+		(start 112.679998 86.878865)
+		(end 112.679998 86.392509)
 		(width 0.252)
 		(layer "F.Cu")
@@
 	)
 	(segment
-		(start 112.679998 86.878865)
-		(end 112.679998 86.392509)
+		(start 113.625998 87.135687)
+		(end 115.034313 87.135687)
 		(width 0.252)
 		(layer "F.Cu")
@@
 	)
 	(segment
-		(start 115.404311 87.135687)
-		(end 115.9 86.639998)
+		(start 115.034313 87.135687)
+		(end 115.530002 86.639998)
 		(width 0.252)
 		(layer "F.Cu")
@@
 	)
 	(segment
-		(start 114.315176 85.635687)
-		(end 115.210863 84.74)
+		(start 115.57 84.74)
+		(end 115.9 84.74)
 		(width 0.252)
 		(layer "F.Cu")
@@
 	)
 	(segment
-		(start 114.571998 86.378865)
-		(end 114.571998 85.892509)
+		(start 114.674313 85.635687)
+		(end 115.57 84.74)
 		(width 0.252)
 		(layer "F.Cu")
@@
 	)
 	(segment
-		(start 115.210863 84.74)
-		(end 115.9 84.74)
+		(start 114.571998 86.378865)
+		(end 114.571998 85.892509)
 		(width 0.252)
 		(layer "F.Cu")
@@
 	)
 	(segment
+		(start 114.315176 85.635687)
+		(end 114.674313 85.635687)
+		(width 0.252)
+		(layer "F.Cu")
+		(net "/USBR_D-")
+	)
+	(segment
 		(start 114.315176 86.635687)
 		(end 114.571998 86.378865)
@@
 		(polygon
 			(pts
-				(xy 105 70) (xy 160 70) (xy 160 100) (xy 105 100)
+				(xy 105 70) (xy 160 70) (xy 160 101.98) (xy 105 101.98)
 			)
 		)
@@
 		)
 	)
+	(generated
+		(type tuning_pattern)
+		(name "Tuning Pattern")
+		(layer "F.Cu")
+		(base_line
+			(pts
+				(xy 121.770665 85.27) (xy 122.910665 85.27)
+			)
+		)
+		(base_line_coupled
+			(pts
+				(xy 120.539528 84.74) (xy 120.552933 84.74)
+			)
+		)
+		(corner_radius_percent 80)
+		(end
+			(xy 122.910665 85.27)
+		)
+		(initial_side "right")
+		(is_time_domain no)
+		(last_diff_pair_gap 0.18)
+		(last_netname "D+")
+		(last_status "too_short")
+		(last_track_width 0.2)
+		(last_tuning_length -0.00131)
+		(max_amplitude 0.24)
+		(min_amplitude 0.2)
+		(min_spacing 0.4)
+		(origin
+			(xy 121.770665 85.27)
+		)
+		(override_custom_rules no)
+		(rounded no)
+		(single_sided no)
+		(target_delay 1000000)
+		(target_delay_max 1000000)
+		(target_delay_min 0)
+		(target_length 1000000)
+		(target_length_max 1000000)
+		(target_length_min 0)
+		(target_skew 0.7)
+		(target_skew_max 0.8)
+		(target_skew_min 0.6)
+		(tuning_mode "diff_pair_skew")
+		(members "32676265-239a-4357-ab27-14398a791c28" "5fde06bc-3419-4844-bf7b-a0a8abdaa12d"
+			"7820ca26-543a-4a03-94a0-f3129e40f4d0" "8ad08d94-1866-4837-bc0c-7ad59239cbe4"
+		)
+	)
