File: feather-SAMD21&WD.kicad_sch (KiCad schematic)
At the start: 42 parts, among them J1 left_header, J10 reset_enable, J2 Batt_header, J3 right_header, J5 16P_USB_C, J6 JumperSET0, J8 JumperSET1, J9 JumperSET2, SW3 SW_Push, U1 ATSAMD21G18A-M, U2 AMS1117-3.3, U3 MAX6369, U5 USBLC6-2SC6

Commit message: minor changes
Parts:
- removed C8, C9: 22u, Capacitor_SMD:C_0805_2012Metric_Pad1.18x1.45mm_HandSolder, symbol Device:C_Small
- removed D2: LED, LED_SMD:LED_0805_2012Metric_Pad1.15x1.40mm_HandSolder, symbol Device:LED
- removed R10: 2k2, Resistor_SMD:R_0805_2012Metric_Pad1.20x1.40mm_HandSolder, symbol Device:R
- removed U2: AMS1117-3.3, Package_TO_SOT_SMD:SOT-223-3_TabPin2, symbol Regulator_Linear:AMS1117-3.3
Other:
- note removed: "3.3v LDO"
- moved on the sheet: C15, C16, C17, C?, FB1, H1, H2, H3, H4, J10, J2, J5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

Commit message: layout done, few sch changes
Parts:
- removed C15: 10n, Capacitor_SMD:C_0805_2012Metric_Pad1.18x1.45mm_HandSolder, symbol Device:C_Small
- removed C16, C17: 1u, Capacitor_SMD:C_0805_2012Metric_Pad1.18x1.45mm_HandSolder, symbol Device:C_Small
- removed FB1: FerriteBead, Inductor_SMD:L_0805_2012Metric_Pad1.05x1.20mm_HandSolder, symbol Device:FerriteBead
- removed H3, H4: MountingHole_Pad, MountingHole:MountingHole_2.2mm_M2_Pad, symbol Mechanical:MountingHole_Pad
- removed L2: RED, Adafruit Feather M0 Express:CHIPLED_0805_NOOUTLINE, symbol Adafruit Feather M0 Express-eagle-import:LED0805_NOOUTLINE
- removed R9: 2.2K, Adafruit Feather M0 Express:0603-NO, symbol Adafruit Feather M0 Express-eagle-import:RESISTOR_0603_NOOUT
- removed TP8: TestPoint_Small, TestPoint:TestPoint_Pad_D1.5mm, symbol Connector:TestPoint_Small
- added C7, C8: 22pf, Capacitor_SMD:C_0805_2012Metric_Pad1.18x1.45mm_HandSolder, symbol Device:C_Small
- added C9: 1u, Capacitor_SMD:C_0805_2012Metric_Pad1.18x1.45mm_HandSolder, symbol Device:C_Small
- added D1: LED, LED_SMD:LED_0805_2012Metric, symbol Device:LED
- added H3, H4: MountingHole, MountingHole:MountingHole_2.5mm, symbol Mechanical:MountingHole
- added R8: 2k2, Resistor_SMD:R_0805_2012Metric_Pad1.20x1.40mm_HandSolder, symbol Device:R_Small
- added X1: 32.768, Crystal:Crystal_SMD_3215-2Pin_3.2x1.5mm, symbol Device:Crystal
- J5: renamed from J3; footprint (none) -> Connector_PinHeader_2.54mm:PinHeader_1x12_P2.54mm_Vertical
- gave numbers to parts that had none: 4
- renumbered C4 to C1, C5 to C2, J6 to J1, J8 to J2, J9 to J3, J1 to J4, J2 to J6, J10 to J7, J5 to J8, R4 to R1, R5 to R2, R7 to R3, R6 to R4, R8 to R5, R13 to R6, R14 to R7, SW3 to SW1, TP10 to TP2, U3 to U1, U5 to U2, U1 to U3
Connections:
- net +3.3VA is gone; now on net +3.3V: U3.6 (VDDANA)
- net EP is gone; now on net GND: U3.49 (EP)
- net +3.3V: no longer U3.43 (VDDCORE)
- net D13: now also R8.1
- net GND: now also C7.1, C8.2, C9.1, D1.1 (K)
- net at U3.1 (PA00): now also C7.2, X1.2
- net at U3.2 (PA01): now also C8.1, X1.1
- new net: C9.2, U3.43 (VDDCORE)
- new net: D1.2 (A), R8.2
- no-connect marks 2 -> 3
Other:
- note added: "HSE osc"
- note removed: "Filtering for 3.3VA"

Commit message: rev one, routing done
Connections:
- net A0: no longer U1.1 (WDI)
- net D1: now also U1.1 (WDI)
Changed lines of the file:
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@@
-		)
-	)
-	(global_label "A0"
-		(shape bidirectional)
-		(at 62.23 170.18 180)
-		(fields_autoplaced yes)
-		(effects
-			(font
-				(size 1.2446 1.2446)
-			)
-			(justify right)
-		)
-		(property "Intersheetrefs" "${INTERSHEET_REFS}"
-			(at 55.9637 170.18 0)
-			(hide yes)
-			(show_name no)
-			(do_not_autoplace no)
-			(effects
-				(font
-					(size 1.27 1.27)
-				)
-				(justify right)
-			)
 		)
 	)
@@
 			(hide yes)
 			(show_name no)
+			(do_not_autoplace no)
+			(effects
+				(font
+					(size 1.27 1.27)
+				)
+				(justify right)
+			)
+		)
+	)
+	(global_label "D1"
+		(shape bidirectional)
+		(at 62.23 170.18 180)
+		(fields_autoplaced yes)
+		(effects
+			(font
+				(size 1.2446 1.2446)
+			)
+			(justify right)
+		)
+		(property "Intersheetrefs" "${INTERSHEET_REFS}"
+			(at 55.7859 170.18 0)
+			(hide yes)
+			(show_name no)

Commit message: V3 schematic updated
Parts:
- removed C6: 100n, Capacitor_SMD:C_0805_2012Metric_Pad1.18x1.45mm_HandSolder, symbol Device:C_Small
- added C10, C11: 22u, Capacitor_SMD:C_0805_2012Metric_Pad1.18x1.45mm_HandSolder, symbol Device:C_Small
- added C12: C, Capacitor_SMD:C_0805_2012Metric_Pad1.18x1.45mm_HandSolder, symbol Device:C_Small
- added C13: 10n, Capacitor_SMD:C_0805_2012Metric_Pad1.18x1.45mm_HandSolder, symbol Device:C_Small
- added C9: 4.7u, Capacitor_SMD:C_0805_2012Metric_Pad1.18x1.45mm_HandSolder, symbol Device:C_Small
- added D2, D6: LED, LED_SMD:LED_0805_2012Metric_Pad1.15x1.40mm_HandSolder, symbol Device:LED
- added D3: D_Schottky, Diode_SMD:D_SOD-123, symbol Device:D_Schottky
- added D4: LED, LED_SMD:LED_0805_2012Metric, symbol Device:LED
- added J10: monostable bypass jumper, Connector_PinHeader_2.54mm:PinHeader_1x02_P2.54mm_Vertical, symbol Connector:Conn_01x02_Pin
- added J9: wd_pwr_jumper, Connector_PinHeader_2.54mm:PinHeader_1x02_P2.54mm_Vertical, symbol Connector:Conn_01x02_Pin
- added R10, R14, R15: 2k2, Resistor_SMD:R_0805_2012Metric_Pad1.20x1.40mm_HandSolder, symbol Device:R
- added R11, R12: 100k, Resistor_SMD:R_0805_2012Metric_Pad1.20x1.40mm_HandSolder, symbol Device:R
- added R13: Rprog, Resistor_SMD:R_0805_2012Metric_Pad1.20x1.40mm_HandSolder, symbol Device:R_Small
- added R16: R, Resistor_SMD:R_0805_2012Metric_Pad1.20x1.40mm_HandSolder, symbol Device:R
- added R9: 2k2, Resistor_SMD:R_0805_2012Metric_Pad1.20x1.40mm_HandSolder, symbol Device:R_Small
- added U4, U6: AP2112K-3.3, Package_TO_SOT_SMD:SOT-23-5, symbol Regulator_Linear:AP2112K-3.3
- added U5: MCP73832-2-OT, Package_TO_SOT_SMD:SOT-23-5, symbol Battery_Management:MCP73832-2-OT
- added U7: LM555xMM, Package_SO:VSSOP-8_3x3mm_P0.65mm, symbol Timer:LM555xMM
- H1, H2: footprint MountingHole:MountingHole_2.2mm_M2_Pad -> Library:feather_mounting hole M2.5
- H3, H4: footprint MountingHole:MountingHole_2.5mm -> Library:feather_mounting hole (no pad)
- J1, J2, J3: footprint Connector_PinHeader_2.54mm:PinHeader_1x02_P2.54mm_Vertical -> Jumper:SolderJumper-2_P1.3mm_Open_RoundedPad1.0x1.5mm
- renumbered C7 to C6, C8 to C7, C9 to C8
Connections:
- net +BATT: now also C9.1, D3.2 (A), R11.2, U5.3 (V_{BAT})
- net GND: now also C10.2, C11.2, C12.2, C13.1, C9.2, R10.1, R12.1, R13.1, R14.1, U4.2 (GND), U5.2 (V_{SS}), U6.2 (GND), U7.1 (GND)
- net VBUS: now also C10.1, D3.1 (K), D4.1 (K), R15.2, U4.1 (VIN), U5.4 (V_{DD})
- net ~{RESET}: no longer J7.1 (Pin_1), R5.2
- net +3.3V renamed +3.3Vmcu
- net +3.3Vmcu: now also D6.2 (A), U6.5 (VOUT); no longer C2.1, J1.1 (Pin_1), J2.1 (Pin_1), J3.1 (Pin_1), J4.15 (Pin_15), R5.1, U1.8 (VCC)
- net RXLED renamed batt_ADC
- net batt_ADC: now also R11.1, R12.2
- net TXLED renamed ldoEN
- net ldoEN: now also J10.1 (Pin_1), U6.3 (EN), U7.3 (OUT)
- new net: D4.2 (A), R9.2
- new net: R15.1, U4.3 (EN)
- new net: R13.2, U5.5 (PROG)
- new net: D2.1 (K), R10.2
- new net: D6.1 (K), R14.2
- new net: R9.1, U5.1 (STAT)
- new net: C13.2, U7.5 (CONT)
- new net: C12.1, U7.6 (THRES)
- new net: R16.1, U7.7 (DISCH)
- new net +3.3Vsys: C11.1, D2.2 (A), J1.1 (Pin_1), J2.1 (Pin_1), J3.1 (Pin_1), J4.15 (Pin_15), J9.1 (Pin_1), U4.5 (VOUT), U6.1 (VIN)
- new net +3.3Vwd: C2.1, J9.2 (Pin_2), R16.2, R5.1, U1.8 (VCC), U7.4 (~{RST}), U7.8 (VCC)
- new net WDO: J10.2 (Pin_2), J7.1 (Pin_1), R5.2, U7.2 (TRIG)
- no-connect marks 3 -> 7
Other:
- note added: "3.3v mcu LDO"
- note added: "3.3v system LDO"
- note added: "Ireg(mA) = 1000/Rprog(kohms) 10k -> 100mA"
- note added: "MCU"
- note added: "T(monostable)= 1.1*R*C"
- note added: "WatchDog System"
- note added: "battery ADC (PB03) (AIN 11)"
- note added: "battery charger"
- note added: "external supply (Buck-system)"
- note added: "good value for 0.5s -> R= 100k, C= 4.7u"
- note added: "monostable - 555"
- moved on the sheet: C1, C2, C3, C4, C5, C6, C7, C8, D1, H1, H2, H3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

Commit message: v3 layout done
Parts:
- added TP1, TP10, TP11, TP12, TP13, TP14, TP15, TP16, TP17, TP3, TP4, TP5, TP6, TP7, TP8, TP9: TestPoint_Small, TestPoint:TestPoint_Pad_D1.5mm, symbol Connector:TestPoint_Small
- J10: footprint Connector_PinHeader_2.54mm:PinHeader_1x02_P2.54mm_Vertical -> Jumper:SolderJumper-2_P1.3mm_Open_Pad1.0x1.5mm
- J7, J9: footprint Connector_PinHeader_2.54mm:PinHeader_1x02_P2.54mm_Vertical -> Jumper:SolderJumper-2_P1.3mm_Open_RoundedPad1.0x1.5mm
Connections:
- net +3.3Vmcu: now also TP6.1; no longer R4.2
- net +3.3Vsys: now also R4.2, TP5.1
- net +3.3Vwd: now also TP4.1
- net +BATT: now also TP7.1
- net A0: now also U1.1 (WDI), TP3.1
- net AREF: now also TP17.1
- net D+: now also TP15.1
- net D-: now also TP16.1
- net D1: no longer U1.1 (WDI)
- net EN: now also R15.1, U4.3 (EN)
- net GND: now also TP9.1
- net VBUS: now also TP13.1; no longer TP2.1
- net WDO: now also TP2.1
- net batt_ADC: now also TP14.1
- net ldoEN: now also TP8.1
- net ~{RESET}: now also TP1.1
- net at R9.1, U5.1 (STAT): now also TP12.1
- net at C12.1, U7.6 (THRES): now also TP10.1
- net at R16.1, U7.7 (DISCH): now also TP11.1

Commit message: final changes, everythings done
Connections:
- net A0: no longer TP3.1, U1.1 (WDI)
- net D1: now also TP3.1, U1.1 (WDI)
Changed lines of the file:
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@@
+		)
+	)
+	(global_label "D1"
+		(shape bidirectional)
+		(at 350.52 175.26 180)
+		(fields_autoplaced yes)
+		(effects
+			(font
+				(size 1.2446 1.2446)
+			)
+			(justify right)
+		)
+		(property "Intersheetrefs" "${INTERSHEET_REFS}"
+			(at 344.0759 175.26 0)
+			(hide yes)
+			(show_name no)
+			(do_not_autoplace no)
+			(effects
+				(font
+					(size 1.27 1.27)
+				)
+				(justify right)
+			)
 		)
 	)
@@
 			(hide yes)
 			(show_name no)
-			(do_not_autoplace no)
-			(effects
-				(font
-					(size 1.27 1.27)
-				)
-				(justify right)
-			)
-		)
-	)
-	(global_label "A0"
-		(shape bidirectional)
-		(at 350.52 175.26 180)
-		(fields_autoplaced yes)
-		(effects
-			(font
-				(size 1.2446 1.2446)
-			)
-			(justify right)
-		)
-		(property "Intersheetrefs" "${INTERSHEET_REFS}"
-			(at 344.2537 175.26 0)
-			(hide yes)
-			(show_name no)

Commit message: finishing touches
Connections:
- no-connect marks 7 -> 4

Commit message: minor changes
Parts:
- removed TP12, TP13, TP15, TP16, TP17, TP3, TP5, TP7, TP9: TestPoint_Small, TestPoint:TestPoint_Pad_D1.5mm, symbol Connector:TestPoint_Small
- removed U1: MAX6369, Package_TO_SOT_SMD:SOT-23-8, symbol Power_Supervisor:MAX6369
- added U8: MAX6373, Package_TO_SOT_SMD:SOT-23-8, symbol Power_Supervisor:MAX6373
- C2: value C_Small -> 100n
- C6, C7: value 22pf -> 12.5pf
- D3: value D_Schottky -> D_Schottky(BAT43W)
- renumbered TP14 to TP3, TP11 to TP5, TP10 to TP7
Connections:
- net +3.3Vwd: now also U8.8 (VCC)
- net D1: now also U8.1 (WDI)
- net GND: now also U8.2 (GND)
- net SET0: now also U8.4 (SET0)
- net SET1: now also U8.5 (SET1)
- net SET2: now also U8.6 (SET2)
- net at J7.2 (Pin_2): now also U8.7 (~{WDO})
